File: differential-buffer-quadchannel.brd (EAGLE design)
At the start: 50.8 x 120.7 mm, 56 parts, among them U1 AD8421, U2 AD8421, U3 AD8421, U4 AD8421

Commit message: Added part numbers
Parts:
- C17, C18: value (none) -> 220uF
- R10, R2, R4, R7: value 10k -> 1M
- RG0, RG1, RG2, RG3: value (none) -> DNP

Commit message: changed RA BNC to vertical
Parts:
- IN_CH0, IN_CH1, IN_CH2, IN_CH3: value BNC-H -> BNC-V; device Eurocard-HV-piezo-driver:BNC90 -> connector-jqi:BNC-V
- OUT_CH0, OUT_CH1, OUT_CH2, OUT_CH3: value BNC-H -> BNC-V; device connector-jqi:BNC90 -> connector-jqi:BNC-V
- moved IN_CH0 0.76 mm to (-17.3, 16.5)
- moved IN_CH1 0.76 mm to (-17.3, -8.89)
- moved IN_CH2 0.76 mm to (-17.3, -34.3)
- moved IN_CH3 0.76 mm to (-17.3, -59.7)
- turned OUT_CH0 to 270 degrees
- turned OUT_CH1 to 270 degrees
- turned OUT_CH2 to 270 degrees
- turned OUT_CH3 to 270 degrees
Routing:
- net N$8: track 3.57 -> 8.65 mm
- net N$24: track 3.57 -> 8.65 mm
- net N$16: track 3.57 -> 8.65 mm
- net N$1: track 3.57 -> 8.65 mm
- net N$56: track 8.47 -> 13.3 mm
- net N$23: track 10.8 -> 15.5 mm
- net N$6: track 8.47 -> 13.0 mm
- net N$22: track 8.47 -> 13.0 mm
- net N$7: track 10.8 -> 15.1 mm
- net N$57: track 10.8 -> 15.1 mm
- net N$15: track 10.8 -> 15.1 mm
- net N$14: track 8.47 -> 12.8 mm
